File: mainboard/mainboard.kicad_sch (KiCad schematic)
At the start: 25 parts, among them J1 Conn_01x04, J2 Conn_01x04, J3 Conn_01x04, J4 Conn_01x04, J5 Conn_01x04, J6 Conn_01x04, J7 Conn_01x04, J8 Conn_01x04, Q1 AO3400A, Q2 AO3400A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

Commit message: feat: finish the layout of mainboard
Parts:
- added H1, H2, H3, H4: MountingHole_5.3mm_M5, MountingHole:MountingHole_5.3mm_M5, symbol Mechanical:MountingHole
- added J5: (no value), symbol Connector_Generic:Conn_01x04
- R1: value (none) -> 1k; footprint (none) -> Resistor_SMD:R_1206_3216Metric_Pad1.30x1.75mm_HandSolder
- R2, R4, R6: footprint (none) -> Resistor_SMD:R_1206_3216Metric_Pad1.30x1.75mm_HandSolder
- renumbered J5 to J6, J6 to J7, J7 to J8, J8 to J9
Connections:
- net MISO: now also J5.3 (Pin_3)
- net MOSI: now also J5.2 (Pin_2)
- net SCK: now also J5.4 (Pin_4)
- net cs5: now reaches U2.13 (~D10/A10)
- net cs5: now also J5.1 (Pin_1)
- no-connect marks 13 -> 12
